Commit message: add gripper on ur5

File: universal_robot/ur_description/urdf/inc/ur_transmissions.xacro (robot description, xacro)
@@ -61,4 +61,22 @@
       </actuator>
     </transmission>
+    <transmission name="${prefix}hande_right_finger_trans">
+      <type>transmission_interface/SimpleTransmission</type>
+      <joint name="${prefix}hande_right_finger_joint">
+        <hardwareInterface>${hw_interface}</hardwareInterface>
+      </joint>
+      <actuator name="${prefix}hande_right_finger_motor">
+        <mechanicalReduction>1</mechanicalReduction>
+      </actuator>
+    </transmission>
+    <transmission name="${prefix}hande_left_finger_trans">
+      <type>transmission_interface/SimpleTransmission</type>
+      <joint name="${prefix}hande_left_finger_joint">
+        <hardwareInterface>${hw_interface}</hardwareInterface>
+      </joint>
+      <actuator name="${prefix}hande_left_finger_motor">
+        <mechanicalReduction>1</mechanicalReduction>
+      </actuator>
+    </transmission>
   </xacro:macro>
 </robot>

File: universal_robot/ur_description/urdf/ur5.xacro (robot description, xacro)
@@ -15,4 +15,5 @@
   -->
   <xacro:include filename="$(find ur_description)/urdf/inc/ur5_macro.xacro"/>
+  <xacro:include filename="$(find ur_description)/urdf/robotiq_hande_gripper.urdf.xacro" />
   <xacro:ur5_robot prefix="" />
 </robot>
